File: hw/esp-lamp.kicad_pcb (KiCad board)
At the start: 2 copper layers, 3 parts, among them U1 AMS1117-3.3, U2 ESP32-WROOM-32, U3 LC12S

Commit message: finalize pcb
Parts:
- added C1: 22uF, Capacitor_SMD:C_0603_1608Metric_Pad1.08x0.95mm_HandSolder, F.Cu at (122.8, 98.0)
- added C10: 10uF, Capacitor_SMD:C_0603_1608Metric_Pad1.08x0.95mm_HandSolder, F.Cu at (127.8, 93.9)
- added C11: 100nF, Capacitor_SMD:C_0603_1608Metric_Pad1.08x0.95mm_HandSolder, F.Cu at (127.8, 92.3)
- added C2: 22uF, Capacitor_SMD:C_0603_1608Metric_Pad1.08x0.95mm_HandSolder, F.Cu at (126.4, 104.0)
- added C3: 100nF, Capacitor_SMD:C_0603_1608Metric_Pad1.08x0.95mm_HandSolder, F.Cu at (151.3, 98.1)
- added C4: 10uF, Capacitor_SMD:C_0603_1608Metric_Pad1.08x0.95mm_HandSolder, F.Cu at (151.7, 105.5)
- added C5: 100n, Capacitor_SMD:C_0603_1608Metric_Pad1.08x0.95mm_HandSolder, F.Cu at (152.3, 109.8)
- added C6: 1nF, Capacitor_SMD:C_0603_1608Metric_Pad1.08x0.95mm_HandSolder, B.Cu at (131.6, 84.2)
- added C7: 1nF, Capacitor_SMD:C_0603_1608Metric_Pad1.08x0.95mm_HandSolder, B.Cu at (137.2, 83.6)
- added C8: 1nF, Capacitor_SMD:C_0603_1608Metric_Pad1.08x0.95mm_HandSolder, B.Cu at (128.4, 116.1)
- added C9: 1nF, Capacitor_SMD:C_0603_1608Metric_Pad1.08x0.95mm_HandSolder, B.Cu at (139.6, 117.5)
- added D1: LED, LED_SMD:LED_0805_2012Metric_Pad1.15x1.40mm_HandSolder, F.Cu at (134.0, 100.0)
- added D2: 1N4148, Diode_SMD:D_SOD-128, F.Cu at (122.4, 95.2)
- added J1: Screw_Terminal_01x02, TerminalBlock_Phoenix:TerminalBlock_Phoenix_MPT-0,5-2-2.54_1x02_P2.54mm_Horizontal, F.Cu at (147.9, 78.8)
- added J2: Expand, Connector_PinHeader_2.54mm:PinHeader_2x04_P2.54mm_Vertical, F.Cu at (144.5, 88.2)
- added J3: JTAG, Connector_PinHeader_2.54mm:PinHeader_2x04_P2.54mm_Vertical, F.Cu at (115.9, 90.5)
- added J4: Serial, Connector_PinHeader_2.54mm:PinHeader_1x03_P2.54mm_Vertical, F.Cu at (131.5, 125.4)
- added J5: USB_C_Receptacle_USB2.0, Connector_USB:USB_C_Receptacle_HRO_TYPE-C-31-M-12, B.Cu at (134.0, 73.0)
- added R1: 6k8, Resistor_SMD:R_0603_1608Metric_Pad0.98x0.95mm_HandSolder, B.Cu at (131.4, 90.6)
- added R10: 6k8, Resistor_SMD:R_0603_1608Metric_Pad0.98x0.95mm_HandSolder, F.Cu at (135.2, 95.4)
- added R11: 470, Resistor_SMD:R_0603_1608Metric_Pad0.98x0.95mm_HandSolder, B.Cu at (137.2, 87.6)
- added R12: 470, Resistor_SMD:R_0603_1608Metric_Pad0.98x0.95mm_HandSolder, B.Cu at (128.4, 111.5)
- added R13: 470, Resistor_SMD:R_0603_1608Metric_Pad0.98x0.95mm_HandSolder, B.Cu at (139.6, 112.4)
- added R14: 100, Resistor_SMD:R_0603_1608Metric_Pad0.98x0.95mm_HandSolder, F.Cu at (130.4, 99.9)
- added R15: 5k1, Resistor_SMD:R_0603_1608Metric_Pad0.98x0.95mm_HandSolder, F.Cu at (132.7, 73.8)
- added R16: 5k1, Resistor_SMD:R_0603_1608Metric_Pad0.98x0.95mm_HandSolder, F.Cu at (135.2, 73.8)
- added R2: 100, Resistor_SMD:R_0603_1608Metric_Pad0.98x0.95mm_HandSolder, B.Cu at (131.4, 89.0)
- added R3: 100, Resistor_SMD:R_0603_1608Metric_Pad0.98x0.95mm_HandSolder, F.Cu at (132.5, 106.8)
- added R4: 100, Resistor_SMD:R_0603_1608Metric_Pad0.98x0.95mm_HandSolder, F.Cu at (132.5, 108.4)
- added R5: 100, Resistor_SMD:R_0603_1608Metric_Pad0.98x0.95mm_HandSolder, F.Cu at (132.5, 105.2)
- added R6: 100, Resistor_SMD:R_0603_1608Metric_Pad0.98x0.95mm_HandSolder, F.Cu at (132.5, 95.6)
- added R7: 470, Resistor_SMD:R_0603_1608Metric_Pad0.98x0.95mm_HandSolder, B.Cu at (133.4, 84.2)
- added R8: 6k8, Resistor_SMD:R_0603_1608Metric_Pad0.98x0.95mm_HandSolder, F.Cu at (136.8, 95.4)
- added R9: 6k8, Resistor_SMD:R_0603_1608Metric_Pad0.98x0.95mm_HandSolder, F.Cu at (138.4, 95.4)
- added REF**: MountingHole_2.2mm_M2, MountingHole:MountingHole_2.2mm_M2, F.Cu at (143.0, 125.0)
- added REF**: MountingHole_2.2mm_M2, MountingHole:MountingHole_2.2mm_M2, F.Cu at (142.0, 75.0)
- added REF**: MountingHole_2.2mm_M2, MountingHole:MountingHole_2.2mm_M2, F.Cu at (125.0, 125.0)
- added REF**: MountingHole_2.2mm_M2, MountingHole:MountingHole_2.2mm_M2, F.Cu at (126.0, 75.0)
- added SW1: RESET, Button_Switch_THT:SW_PUSH_6mm_H4.3mm, F.Cu at (116.8, 78.8)
- added SW2: X-BOOT, Button_Switch_THT:SW_PUSH-12mm_Wuerth-430476085716, F.Cu at (127.8, 82.5)
- added SW3: A, Button_Switch_THT:SW_PUSH-12mm_Wuerth-430476085716, F.Cu at (118.8, 113.7)
- added SW4: B, Button_Switch_THT:SW_PUSH-12mm_Wuerth-430476085716, F.Cu at (136.8, 113.7)
- U2, U3: moved to B.Cu
- moved U2 114.8 mm to (144.6, 100.0), turned to 90 degrees
- moved U1 82.8 mm to (120.8, 102.8), turned to 180 degrees
- moved U3 58.9 mm to (128.9, 93.6), turned to -90 degrees
Routing:
- net 3V3: track 0.00 -> 96.6 mm, vias 0 -> 12
- net TXD: track 0.00 -> 44.6 mm, vias 0 -> 1
- net Net-(U2-IO4): track 0.00 -> 43.1 mm, vias 0 -> 2
- net Vin: track 0.00 -> 41.0 mm, vias 0 -> 1
- net Net-(J3-Pin_4): track 0.00 -> 39.9 mm
- net EN: track 0.00 -> 39.6 mm, vias 0 -> 2
- net RXD: track 0.00 -> 39.2 mm, vias 0 -> 1
- net Net-(J3-Pin_3): track 0.00 -> 31.4 mm
- net Net-(J3-Pin_5): track 0.00 -> 30.7 mm
- net UA: track 0.00 -> 27.3 mm, vias 0 -> 1
- net UB: track 0.00 -> 25.5 mm, vias 0 -> 1
- net UC: track 0.00 -> 23.0 mm, vias 0 -> 1
- net LSC_CS: track 0.00 -> 22.7 mm, vias 0 -> 2
- net Net-(U2-IO2): track 0.00 -> 21.4 mm, vias 0 -> 1
- net LSC_SET: track 0.00 -> 21.4 mm, vias 0 -> 2
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- added copper zone on B.Cu, net 3V3
- added copper zone on F.Cu, net 3V3
- added copper zone on B.Cu, net GND
- added copper zone on F.Cu, net GND
Other:
- board outline added: 40 x 60 mm
- board text added: "+ -"
- board text added: "AUX IO"
- board text added: "BNT-B"
- board text added: "BTN-A"
- board text added: "BTN-XBoot"
- board text added: "ESP-LAMP"
- board text added: "G Tx Rx"
- board text added: "JTAG"
- board text added: "PWR"
- board text added: "RST"
- board text added: "Vanek 2024"
