File: hw/esp-lamp.kicad_sch (KiCad schematic)
At the start: 38 parts, among them J1 Screw_Terminal_01x02, J2 Expand, J3 JTAG, J4 Serial, SW1 RESET, SW2 X-BOOT, SW3 A, SW4 B, U1 AMS1117-3.3, U2 ESP32-WROOM-32, U3 LC12S

Commit message: finalize pcb
Parts:
- added J5: USB_C_Receptacle_USB2.0, Connector_USB:USB_C_Receptacle_HRO_TYPE-C-31-M-12, symbol Connector:USB_C_Receptacle_USB2.0
- added R15, R16: 5k1, Resistor_SMD:R_0603_1608Metric_Pad0.98x0.95mm_HandSolder, symbol Device:R
- C1, C10, C11, C2, C3, C4, C5, C6, C7, C8, C9: footprint (none) -> Capacitor_SMD:C_0603_1608Metric_Pad1.08x0.95mm_HandSolder
- D1: footprint (none) -> LED_SMD:LED_0805_2012Metric_Pad1.15x1.40mm_HandSolder
- D2: footprint Diode_THT:D_DO-35_SOD27_P7.62mm_Horizontal -> Diode_SMD:D_SOD-128
- J1: footprint (none) -> TerminalBlock_Phoenix:TerminalBlock_Phoenix_MPT-0,5-2-2.54_1x02_P2.54mm_Horizontal
- J2, J3: footprint (none) -> Connector_PinHeader_2.54mm:PinHeader_2x04_P2.54mm_Vertical
- J4: footprint (none) -> Connector_PinHeader_2.54mm:PinHeader_1x03_P2.54mm_Vertical
- R1, R10, R11, R12, R13, R14, R2, R3, R4, R5, R6, R7, R8, R9: footprint (none) -> Resistor_SMD:R_0603_1608Metric_Pad0.98x0.95mm_HandSolder
- SW1: footprint (none) -> Button_Switch_THT:SW_PUSH_6mm_H4.3mm
- SW2, SW3, SW4: footprint (none) -> Button_Switch_THT:SW_PUSH-12mm_Wuerth-430476085716
Connections:
- net GND: now also R14.1, J5.A1 (GND), J5.A12 (GND), J5.B1 (GND), J5.B12 (GND), J5.S1 (SHIELD), R15.2, R16.2; no longer D1.1 (K)
- net Vin: now reaches D2.2 (A), J1.2 (Pin_2)
- net Vin: now also J5.A4 (VBUS), J5.A9 (VBUS), J5.B4 (VBUS), J5.B9 (VBUS)
- net at U2.29 (IO5): now also D1.2 (A); no longer R14.2
- new net: J5.A5 (CC1), R15.1
- new net: J5.B5 (CC2), R16.1
- new net: D1.1 (K), R14.2
- no-connect marks 13 -> 19
Other:
- moved on the sheet: D1, J1, R14
